Commit message: Our 2016 version of walrus repo

File: walrus_description/urdf/boom.urdf.xacro (robot description, xacro)
@@ -1,5 +1,5 @@
 <?xml version="1.0"?>
 <robot xmlns:xacro="http://ros.org/wiki/xacro" name="walrus_boom">
-        <xacro:include filename="$(find walrus_description)/urdf/kinectv2.urdf.xacro" />
+        <xacro:include filename="$(find walrus_description)/urdf/kinect2_centered.urdf.xacro" />
 	<xacro:macro name="walrus_boom" params="parent tf_prefix robot_ns">
 		<!-- Boom base -->
@@ -17,5 +17,5 @@
 			                <box size = "0.08 0.04 0.02"/>
 				</geometry>
-				<material name="green">
+				<material name="black">
 					<color rgba="0 0.8 0 1"/>
 				</material>
@@ -46,5 +46,5 @@
 			                <box size = "0.04 0.04 0.02"/>
 				</geometry>
-				<material name="green">
+				<material name="black">
 					<color rgba="0 0.8 0 1"/>
 				</material>
@@ -85,5 +85,5 @@
 			                <cylinder length="0.5" radius="0.02"/>
 				</geometry>
-				<material name="green">
+				<material name="black">
 					<color rgba="0 0.8 0 1"/>
 				</material>
@@ -126,5 +126,5 @@
 			                <box size = "0.04 0.1 0.02"/>
 				</geometry>
-				<material name="green">
+				<material name="black">
 					<color rgba="0 0.8 0 1"/>
 				</material>
@@ -153,7 +153,8 @@
 		</transmission>
 		<!-- Kinect -->
-		<kinectv2 parent="${tf_prefix}tilt_base" tf_prefix="${tf_prefix}kinect" camera_ns="${robot_ns}/kinect" name="boom_kinect">
+		<!--kinect2 parent="${tf_prefix}tilt_base" tf_prefix="${tf_prefix}kinect" camera_ns="${robot_ns}/kinect" name="boom_kinect"-->
+		<kinect2 parent="${tf_prefix}tilt_base" tf_prefix="${tf_prefix}kinect" name="kinect" >
 			<origin xyz="0 0 0.03" rpy="0 0 0" />
-		</kinectv2>
+		</kinect2>
   	</xacro:macro>
 </robot>

File: walrus_description/urdf/pod.urdf.xacro (robot description, xacro)
@@ -1,4 +1,4 @@
 <?xml version="1.0" encoding="utf-8"?>
-<robot xmlns:xacro="http://ros.org/wiki/xacro" name="walrus_pod">
+<robot xmlns:xacro="http://ros.org/wiki/xacro" name="walrus_pod" machine="walrus">
 	<xacro:macro name="walrus_pod" params="fb lr parent translateX translateY flipY tf_prefix"> <!--fb : front, back ; lr: left, right -->
 		<link name="${tf_prefix}${fb}_${lr}_pod">
@@ -12,5 +12,5 @@
 				<origin xyz="0 0 0" rpy="${M_PI/2 - flipY*M_PI/2} 0 0" />
 				<geometry>
-				  <mesh filename="package://walrus_description/meshes/pod.stl" />
+				  <mesh filename="package://walrus_description/meshes/pod.stl" machine="walrus"/>
 				</geometry>
 				<material name="Red">

Commit message: Added fake boom messages, support for new kinect driver, added the respective m\ odel with correct frames and updated robot.launch accordingly, modified connect\ () fucntion for motors.

File: walrus_description/urdf/boom.urdf.xacro (robot description, xacro)
@@ -154,5 +154,5 @@
 		<!-- Kinect -->
 		<!--kinect2 parent="${tf_prefix}tilt_base" tf_prefix="${tf_prefix}kinect" camera_ns="${robot_ns}/kinect" name="boom_kinect"-->
-		<kinect2 parent="${tf_prefix}tilt_base" tf_prefix="${tf_prefix}kinect" name="kinect" >
+		<kinect2 parent="${tf_prefix}tilt_base" tf_prefix="kinect" name="kinect" >
 			<origin xyz="0 0 0.03" rpy="0 0 0" />
 		</kinect2>

File: walrus_description/urdf/kinect2.urdf.xacro (robot description, xacro)
@@ -5,5 +5,5 @@
 <!-- License: GPLv3+ -->
 <robot xmlns:xacro="http://ros.org/wiki/xacro" name="kinect2">
-  <xacro:macro name="kinect2" params="parent *origin tf_prefix name">
+  <xacro:macro name="kinect2" params="parent *origin tf_prefix">
     <material name="Kinect2Grey">
       <color rgba="0.15 0.15 0.15 1.0"/>
@@ -20,5 +20,5 @@
         <geometry>
           <!-- these meshes were exported in mm, so scale back to m -->
-          <mesh filename="package://walrus_description/meshes/kinect2/kinect2_centered.stl" scale="0.001 0.001 0.001"/>
+          <mesh filename="package://walrus_description/meshes/kinect2/kinect2_origin_on_rgb_optical_frame.stl" scale="0.001 0.001 0.001"/>
         </geometry>
         <material name="Kinect2Grey"/>
