Commit message: better kinect pose, rotatedkinect output 	modified:   walrus_boomboard_driver/src/walrus_boomboard_driver/dummy_boom_state_publisher.cpp 	deleted:    walrus_description/urdf/kinect2.urdf.xacro 	modified:   walrus_description/urdf/kinect2_centered.urdf.xacro

File: walrus_description/urdf/kinect2_centered.urdf.xacro (robot description, xacro)
@@ -26,5 +26,5 @@
     <!-- Joint connecting the ir frame to base frame -->
     <joint name="${tf_prefix}_ir_joint" type="fixed">
-      <origin rpy="0 0 0" xyz="0 0 .025"/>
+      <origin rpy="${-M_PI/2} 0 ${-M_PI/2}" xyz="0 0 .025"/>
       <parent link="${tf_prefix}_base"/>
       <child link="${tf_prefix}_ir_optical_frame"/>
@@ -34,5 +34,5 @@
      <!-- Joint connecting the rgb frame to base frame -->
     <joint name="${tf_prefix}_rgb_joint" type="fixed">
-      <origin rpy="0 0 0" xyz="0 -.100 .025"/>
+      <origin rpy="${-M_PI/2} 0 ${-M_PI/2}" xyz="0 -.100 .025"/>
       <parent link="${tf_prefix}_base"/>
       <child link="${tf_prefix}_rgb_optical_frame"/>
@@ -40,4 +40,5 @@
     <link name="${tf_prefix}_rgb_optical_frame">
     </link>
+	<!--TO DO: add gazebo block from the old file-->
   </xacro:macro>
 </robot>
