Commit message: Fixed pod model and some odometry bugs 	modified:   walrus_boomboard_driver/src/walrus_boomboard_driver/dummy_boom_state_publisher.cpp 	modified:   walrus_bringup/launch/robot.launch 	modified:   walrus_bringup/launch/robot.launch~ 	modified:   walrus_description/urdf/base.urdf.xacro 	modified:   walrus_description/urdf/pod.urdf.xacro 	modified:   walrus_drive_controller/include/walrus_drive_controller/walrus_drive_controller.h 	modified:   walrus_drive_controller/src/odometry.cpp 	modified:   walrus_drive_controller/src/walrus_drive_controller.cpp 	modified:   walrus_system_configuration/upstart.conf

File: walrus_description/urdf/base.urdf.xacro (robot description, xacro)
@@ -131,8 +131,8 @@
       <walrus_center_tread lr="right" parent="${tf_prefix}base_link" translateY="-1" flipY="-1" tf_prefix="${tf_prefix}"/>
       <!-- Pods -->
-      <walrus_pod fb="back" lr="left" parent="${tf_prefix}base_link" translateX="-1" translateY="1" flipY="1" tf_prefix="${tf_prefix}"/>
-      <walrus_pod fb="back" lr="right" parent="${tf_prefix}base_link" translateX="-1" translateY="-1" flipY="-1" tf_prefix="${tf_prefix}"/>
-      <walrus_pod fb="front" lr="left" parent="${tf_prefix}base_link" translateX="1" translateY="1" flipY="1" tf_prefix="${tf_prefix}"/>
-      <walrus_pod fb="front" lr="right" parent="${tf_prefix}base_link" translateX="1" translateY="-1" flipY="-1" tf_prefix="${tf_prefix}"/>
+      <walrus_pod fb="back" lr="left" parent="${tf_prefix}base_link" translateX="-1" translateY="1" flipY="1" rotate="-1.2" tf_prefix="${tf_prefix}"/>
+      <walrus_pod fb="back" lr="right" parent="${tf_prefix}base_link" translateX="-1" translateY="-1" flipY="-1" rotate="0" tf_prefix="${tf_prefix}"/>
+      <walrus_pod fb="front" lr="left" parent="${tf_prefix}base_link" translateX="1" translateY="1" flipY="1" rotate="0" tf_prefix="${tf_prefix}"/>
+      <walrus_pod fb="front" lr="right" parent="${tf_prefix}base_link" translateX="1" translateY="-1" flipY="-1" rotate="0" tf_prefix="${tf_prefix}"/>
       <!-- Cameras -->
       <simple_camera parent="${tf_prefix}base_link" tf_prefix="${tf_prefix}front_camera" camera_ns="${robot_ns}/front_camera" name="front_camera">

File: walrus_description/urdf/pod.urdf.xacro (robot description, xacro)
@@ -1,5 +1,5 @@
 <?xml version="1.0" encoding="utf-8"?>
 <robot xmlns:xacro="http://ros.org/wiki/xacro" name="walrus_pod" machine="walrus">
-	<xacro:macro name="walrus_pod" params="fb lr parent translateX translateY flipY tf_prefix"> <!--fb : front, back ; lr: left, right -->
+	<xacro:macro name="walrus_pod" params="fb lr parent translateX translateY flipY rotate tf_prefix "> <!--fb : front, back ; lr: left, right -->
 		<link name="${tf_prefix}${fb}_${lr}_pod">
 			<inertial>
@@ -10,5 +10,5 @@
 			</inertial>
 			<visual>
-				<origin xyz="0 0 0" rpy="${M_PI/2 - flipY*M_PI/2} 0 0" />
+				<origin xyz="0 0 0" rpy="${M_PI/2 - flipY*M_PI/2} ${rotate*M_PI/2} 0" />
 				<geometry>
 				  <mesh filename="package://walrus_description/meshes/pod.stl" machine="walrus"/>

Commit message: boom parameteres in urdf 	modified:   walrus_description/urdf/base.urdf.xacro 	modified:   walrus_description/urdf/boom.urdf.xacro 	modified:   walrus_description/urdf/boom.urdf.xacro~ 	modified:   walrus_description/urdf/kinect2_centered.urdf.xacro 	modified:   walrus_description/urdf/kinect2_centered.urdf.xacro~

File: walrus_description/urdf/base.urdf.xacro (robot description, xacro)
@@ -131,6 +131,6 @@
       <walrus_center_tread lr="right" parent="${tf_prefix}base_link" translateY="-1" flipY="-1" tf_prefix="${tf_prefix}"/>
       <!-- Pods -->
-      <walrus_pod fb="back" lr="left" parent="${tf_prefix}base_link" translateX="-1" translateY="1" flipY="1" rotate="-1.2" tf_prefix="${tf_prefix}"/>
-      <walrus_pod fb="back" lr="right" parent="${tf_prefix}base_link" translateX="-1" translateY="-1" flipY="-1" rotate="0" tf_prefix="${tf_prefix}"/>
+      <walrus_pod fb="back" lr="left" parent="${tf_prefix}base_link" translateX="-1" translateY="1" flipY="1" rotate="-1.4" tf_prefix="${tf_prefix}"/>
+      <walrus_pod fb="back" lr="right" parent="${tf_prefix}base_link" translateX="-1" translateY="-1" flipY="-1" rotate="0.6" tf_prefix="${tf_prefix}"/>
       <walrus_pod fb="front" lr="left" parent="${tf_prefix}base_link" translateX="1" translateY="1" flipY="1" rotate="0" tf_prefix="${tf_prefix}"/>
       <walrus_pod fb="front" lr="right" parent="${tf_prefix}base_link" translateX="1" translateY="-1" flipY="-1" rotate="0" tf_prefix="${tf_prefix}"/>

File: walrus_description/urdf/boom.urdf.xacro (robot description, xacro)
@@ -30,5 +30,5 @@
 			<parent link="${parent}"/>
 			<child link="${tf_prefix}base"/>
-			<origin xyz="-0.23 0 0.03" rpy="0 0 0" />
+			<origin xyz="-0.40 0 0.1" rpy="0 0 0" />
 		</joint>
 		<!-- Deploy base -->

File: walrus_description/urdf/kinect2_centered.urdf.xacro (robot description, xacro)
@@ -6,5 +6,5 @@
   <xacro:macro name="kinect2" params="parent name *origin tf_prefix">
     <material name="Kinect2Grey">
-      <color rgba="0.15 0.15 0.15 1.0"/>
+      <color rgba="0.10 0.10 0.10 1.0"/>
     </material>
     <!-- Joint connecting the parent to our frame_in -->
@@ -26,5 +26,5 @@
     <!-- Joint connecting the ir frame to base frame -->
     <joint name="${tf_prefix}_ir_joint" type="fixed">
-      <origin rpy="${-M_PI/2} 0 ${-M_PI/2}" xyz="0 0 .025"/>
+      <origin rpy="${-M_PI/2} 0 ${-M_PI/2}" xyz="0 0 -.025"/>
       <parent link="${tf_prefix}_base"/>
       <child link="${tf_prefix}_ir_optical_frame"/>
@@ -34,5 +34,5 @@
      <!-- Joint connecting the rgb frame to base frame -->
     <joint name="${tf_prefix}_rgb_joint" type="fixed">
-      <origin rpy="${-M_PI/2} 0 ${-M_PI/2}" xyz="0 -.100 .025"/>
+      <origin rpy="${-M_PI/2} 0 ${-M_PI/2}" xyz="0 -.100 -.025"/>
       <parent link="${tf_prefix}_base"/>
       <child link="${tf_prefix}_rgb_optical_frame"/>
