Commit message: modified:   walrus_bringup/launch/includes/common.launch.xml 	modified:   walrus_bringup/launch/robot.launch 	modified:   walrus_bringup/launch/robot.launch~ 	modified:   walrus_description/launch/description.launch 	modified:   walrus_description/robots/walrus.urdf.xacro 	modified:   walrus_description/urdf/boom.urdf.xacro 	modified:   walrus_description/urdf/boom.urdf.xacro~

File: walrus_description/robots/walrus.urdf.xacro (robot description, xacro)
@@ -7,4 +7,5 @@
   <property name="tf_prefix" value="$(arg tf_prefix)" />
   <property name="robot_ns" value="$(arg robot_ns)" />
+  <property name="kinect_screw" value="$(arg kinect_screw)" />
   <xacro:walrus tf_prefix="${tf_prefix}" robot_ns="${robot_ns}"/>
   <gazebo>
@@ -29,4 +30,9 @@
     </gazebo>
   </xacro:if>
+  <property name="kinect_screw" value="$(arg kinect_screw)" />
+  <xacro:if value="$(arg hard_kinect)">
+    <xacro:kinect2 parent="${tf_prefix}tilt_base" tf_prefix="kinect" name="kinect" >
+			<origin xyz="5*${kinect_screw} 0 0" rpy="0 0 0" />
+  </xacro:if>
   <xacro:if value="$(arg have_oryx_arm)">
     <xacro:oryx_arm parent="${tf_prefix}base_link" tf_prefix="${tf_prefix}arm/" robot_ns="${robot_ns}/arm"/>

File: walrus_description/urdf/boom.urdf.xacro (robot description, xacro)
@@ -155,5 +155,5 @@
 		<!--kinect2 parent="${tf_prefix}tilt_base" tf_prefix="${tf_prefix}kinect" camera_ns="${robot_ns}/kinect" name="boom_kinect"-->
 		<kinect2 parent="${tf_prefix}tilt_base" tf_prefix="kinect" name="kinect" >
-			<origin xyz="0 0 0.03" rpy="0 0 0" />
+			<origin xyz="0 0 0" rpy="0 0 0" />
 		</kinect2>
   	</xacro:macro>
